File: PCB/MacroBoard.brd (EAGLE design)
At the start: 61 x 81 mm, 44 parts, among them IC1 74AHC1G125DBV, SW1 PEC11, U1 XIAO-RP2040

Commit message: V1.1 update
Parts:
- LED1, LED2, LED3, LED4, LED5, LED6, LED7, LED8, LED9: value WS2812B_SK6812E -> MICROBUILDER_WS2812B_SK6812E; device microbuilder:NEO3535_REVERSE -> MacroBoard:MICROBUILDER_NEO3535_REVERSE
- S1, S2, S3, S4, S5, S6, S7, S8, S9: device adafruit_electromech:KAILH_SOCKET -> MacroBoard:ADAFRUIT_ELECTROMECH_KAILH_SOCKET
- SW1: device adafruit_electromech:PEC11+SWITCH -> MacroBoard:ADAFRUIT_ELECTROMECH_PEC11+SWITCH
- U1: value XIAO-RP2040 -> SEEED-STUDIO-XIAO-SERIES_XIAO-RP2040; device Seeed Studio XIAO Series:XIAO-SAMD21/RP2040-MODULE14P-2.54-21X17.8MM -> MacroBoard:SEEED-STUDIO-XIAO-SERIES_XIAO-SAMD21/RP2040-MODULE14P-2.54-21X17.8MM
- moved IC1 9.16 mm to (11.4, 59.7), turned to 270 degrees
Routing:
- net NEOPIXEL: track 24.1 -> 12.2 mm
- net N$9: track 4.25 -> 9.77 mm
- net +5V: track 249.2 -> 244.3 mm
Other:
- board text added: "V1.1 NOV 2022 palmacas.com"
- board text removed: "V1 JUL 2022 palmacas.com"
