File: PCB/MacroBoard.sch (EAGLE design)
At the start: 43 parts, among them IC1 74AHC1G125DBV, SW1 PEC11, U1 XIAO-RP2040

Commit message: V1.1 update
Parts:
- LED1, LED2, LED3, LED4, LED5, LED6, LED7, LED8, LED9: value WS2812B_SK6812E -> MICROBUILDER_WS2812B_SK6812E; device microbuilder:WS2812B_SK6812E -> MacroBoard:MICROBUILDER_WS2812B_SK6812E
- S1, S2, S3, S4, S5, S6, S7, S8, S9: device adafruit_electromech:KBD_SWITCH_KAILH_SOCKETBOX_JADE_KAILH_SOCKET -> MacroBoard:ADAFRUIT_ELECTROMECH_KBD_SWITCH_KAILH_SOCKETBOX_JADE_KAILH_SOCKET
- SW1: device adafruit_electromech:ENCODER_PLUS_SWITCH_BOURNS_PEC11 -> MacroBoard:ADAFRUIT_ELECTROMECH_ENCODER_PLUS_SWITCH_BOURNS_PEC11
- U1: value XIAO-RP2040 -> SEEED-STUDIO-XIAO-SERIES_XIAO-RP2040; device Seeed Studio XIAO Series:XIAO-RP2040 -> MacroBoard:SEEED-STUDIO-XIAO-SERIES_XIAO-RP2040
